Commit message: Added ultrasonic and depth cam functionality

File: description/camera.xacro (robot description, xacro)
@@ -4,5 +4,5 @@
         <parent link="chassis"/>
         <child link="camera_link"/>
-        <origin xyz="0.276 0 ${chassis_height+0.1}" rpy="0 0.18 0"/>
+        <origin xyz="${chassis_length/2} 0 ${chassis_height+0.17}" rpy="0 0.18 0"/>
     </joint>
     <link name="camera_link">

File: description/depth_camera.xacro (robot description, xacro)
@@ -4,13 +4,29 @@
         <parent link="chassis"/>
         <child link="camera_link"/>
-        <origin xyz="0.305 0 0.08" rpy="0 0 0"/>
+        <origin xyz="${chassis_length} 0 ${chassis_height+0.15}" rpy="0 0.18 0"/>
     </joint>
     <link name="camera_link">
         <visual>
+            <origin xyz="0 0 0.06" rpy="0 0 0"/>
+            <geometry>
+                <box size="0.010 0.10 0.02"/>
+            </geometry>
+            <material name="red"/>
+        </visual>
+        <visual>
+            <origin xyz="0 0 -0.05"/>
+            <geometry>
+                <cylinder radius="0.002" length="0.2"/>
+            </geometry>
+            <material name="black"/>
+        </visual>
+        <collision>
             <geometry>
                 <box size="0.010 0.03 0.03"/>
             </geometry>
-            <material name="red"/>
-        </visual>
+        </collision>
+        <xacro:inertial_box mass="0.05" x="0.010" y="0.03" z="0.03">
+            <origin xyz="0 0 0" rpy="0 0 0"/>
+        </xacro:inertial_box>
     </link>
     <joint name="camera_optical_joint" type="fixed">
@@ -22,12 +38,13 @@
     <gazebo reference="camera_link">
         <material>Gazebo/Red</material>
-        <sensor name="camera" type="depth">
+        <sensor name="rgbd_camera" type="rgbd_camera">
             <pose> 0 0 0 0 0 0 </pose>
             <visualize>true</visualize>
             <update_rate>10</update_rate>
             <camera>
+                <camera_info_topic>rgbd_camera/camera_info</camera_info_topic>
                 <horizontal_fov>1.089</horizontal_fov>
                 <image>
-                    <format>B8G8R8</format>
+                    <format>R8G8B8</format>
                     <width>640</width>
                     <height>480</height>
@@ -38,9 +55,6 @@
                 </clip>
             </camera>
-            <plugin name="camera_controller" filename="libgazebo_ros_camera.so">
-                <frame_name>camera_link_optical</frame_name>
-                <min_depth>0.1</min_depth>
-                <max_depth>100.0</max_depth>
-            </plugin>
+            <topic>rgbd_camera</topic>
+            <gz_frame_id>camera_link_optical</gz_frame_id>
         </sensor>
     </gazebo>

File: description/lidar.xacro (robot description, xacro)
@@ -4,5 +4,5 @@
         <parent link="chassis"/>
         <child link="laser_frame"/>
-        <origin xyz="0.122 0 ${chassis_height+0.02}" rpy="0 0 0"/>
+        <origin xyz="${chassis_length} 0 ${chassis_height+0.24}" rpy="0 0 0"/>
     </joint>
     <link name="laser_frame">
@@ -13,5 +13,5 @@
             <material name="black"/>
         </visual>
-        <visual>
+        <!-- <visual>
             <origin xyz="0 0 -0.05"/>
             <geometry>
@@ -19,5 +19,5 @@
             </geometry>
             <material name="black"/>
-        </visual>
+        </visual> -->
         <collision>
             <geometry>
@@ -30,5 +30,4 @@
     </link>
     <gazebo reference="laser_frame">
-        <material>Gazebo/Black</material>
         <sensor name="laser" type="gpu_lidar">
             <pose> 0 0 0 0 0 0 </pose>

File: description/robot.urdf.xacro (robot description, xacro)
@@ -11,6 +11,7 @@
     </xacro:unless>
     <xacro:include filename="lidar.xacro" />
-    <xacro:include filename="camera.xacro" />
-    <!-- <xacro:include filename="depth_camera.xacro" /> -->
+    <!-- <xacro:include filename="camera.xacro" /> -->
+    <xacro:include filename="depth_camera.xacro" />
+    <xacro:include filename="ultrasonic.xacro" />
     <xacro:include filename="face.xacro" />
 </robot>
